File: receiver/receiver.kicad_sch (KiCad schematic)
At the start: 0 parts

Commit message: devlog 02
Parts:
- added C1: 100nF, symbol Device:C
- added C2: 10uF, symbol Device:C
- added C3: 1uF, symbol Device:C
- added D_ACT: ACT, symbol Device:LED
- added HDR1: DEBUG, symbol Connector_Generic:Conn_01x03
- added J1: USB-C, symbol Connector:USB_C_Receptacle_USB2.0_16P
- added R_ACT: 1k, symbol Device:R
- added R_CC1, R_CC2: 5.1k, symbol Device:R
- added R_EN: 10k, symbol Device:R
- added SW_BOOT: BOOT, symbol Switch:SW_Push
- added SW_RST: RESET, symbol Switch:SW_Push
- added U1: ESP32-S3-WROOM-1, symbol RF_Module:ESP32-S3-WROOM-1
- added U2: AP2112K-3.3, symbol Regulator_Linear:AP2112K-3.3
Connections:
- new net: J1.A1 (GND), J1.A12 (GND), J1.B1 (GND), J1.B12 (GND)
- new net: J1.A4 (VBUS), J1.A9 (VBUS), J1.B4 (VBUS), J1.B9 (VBUS)
- new net: U1.1 (GND), U1.40 (GND), U1.41 (GND)
- no-connect marks 0 -> 2

Commit message: devlog 03
Connections:
- net 3v3: now reaches C2.1
- net 3v3: now also C1.1, R_EN.2, U1.2 (3V3), U2.5 (VOUT)
- net GND: now reaches C2.2
- net GND: now also C1.2, C3.2, D_ACT.1 (K), HDR1.1 (Pin_1), J1.A1 (GND), J1.A12 (GND), J1.B1 (GND), J1.B12 (GND), J1.SH (SHIELD), R_CC1.2, R_CC2.2, SW_BOOT.2, SW_RST.2, U1.1 (GND), U1.40 (GND), U1.41 (GND), U2.2 (GND)
- net CC2: now reaches R_CC2.1
- net CC2: now also J1.B5 (CC2)
- net UART_RX: now reaches HDR1.2 (Pin_2)
- net UART_RX: now also U1.36 (RXD0)
- net UART_TX: now reaches HDR1.3 (Pin_3)
- net UART_TX: now also U1.37 (TXD0)
- net EN_NET: now reaches R_EN.1
- net EN_NET: now also SW_RST.1, U1.3 (EN)
- net VBUS: now reaches U2.1 (VIN)
- net VBUS: now also C3.1, J1.A4 (VBUS), J1.A9 (VBUS), J1.B4 (VBUS), J1.B9 (VBUS), U2.3 (EN)
- net LED_ACT: now reaches R_ACT.1
- net LED_ACT: now also U1.4 (IO4)
- net ACT_A: now reaches R_ACT.2
- net ACT_A: now also D_ACT.2 (A)
- net CC1: now reaches R_CC1.1
- net CC1: now also J1.A5 (CC1)
- net BOOT_NET: now reaches SW_BOOT.1
- net BOOT_NET: now also U1.27 (IO0)
- net USB_DP: now reaches J1.A6 (D+)
- net USB_DP: now also J1.B6 (D+), U1.14 (USB_D+)
- net USB_DN: now reaches J1.A7 (D-)
- net USB_DN: now also J1.B7 (D-), U1.13 (USB_D-)
- no-connect marks 2 -> 32
Other:
- moved on the sheet: C1, C2, HDR1

Commit message: fix stuff
Parts:
- renumbered D_ACT to D1
Changed lines of the file:
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@@
 		(in_pos_files yes)
 		(dnp no)
-		(property "Reference" "D_ACT"
+		(property "Reference" "D1"
 			(at 149.86 116.84 0)
 			(show_name no)
@@
 			(project "receiver"
 				(path "/190c1e52-8c3e-49f8-9174-beae767bddea"
-					(reference "D_ACT")
+					(reference "D1")
 					(unit 1)
 				)
@@
 		)
 	)
+	(symbol
+		(lib_id "power:PWR_FLAG")
+		(at 39.37 111.76 0)
+		(unit 1)
+		(body_style 1)
+		(exclude_from_sim no)
+		(in_bom yes)
+		(on_board yes)
+		(in_pos_files yes)
+		(dnp no)
+		(property "Reference" "#PWR03"
+			(at 39.37 109.22 0)
+			(show_name no)
+			(do_not_autoplace no)
+			(effects
+				(font
+					(size 1.27 1.27)
+				)
+			)
+		)
+		(property "Value" "PWR_FLAG"
+			(at 39.37 114.3 0)
+			(show_name no)
+			(do_not_autoplace no)
+			(effects
+				(font
+					(size 1.27 1.27)
+				)
+			)
+		)
+		(property "Footprint" ""
+			(at 39.37 111.76 0)
+			(hide yes)
+			(show_name no)
+			(do_not_autoplace no)
+			(effects
+				(font
+					(size 1.27 1.27)
+				)
+			)
+		)
+		(property "Datasheet" ""
+			(at 39.37 111.76 0)
+			(hide yes)
+			(show_name no)
+			(do_not_autoplace no)
+			(effects
+				(font
+					(size 1.27 1.27)
+				)
+			)
+		)
+		(property "Description" "Special symbol for telling ERC where power comes from"
+			(at 39.37 111.76 0)
+			(hide yes)
+			(show_name no)
+			(do_not_autoplace no)
+			(effects
+				(font
+					(size 1.27 1.27)
+				)
+			)
+		)
+		(pin "1"
+		)
+		(instances
+			(project "receiver"
+				(path "/190c1e52-8c3e-49f8-9174-beae767bddea"
+					(reference "#PWR03")
+					(unit 1)
+				)
+			)
+		)
+	)
+	(symbol
+		(lib_id "power:PWR_FLAG")
+		(at 39.37 114.3 0)
+		(unit 1)
+		(body_style 1)
+		(exclude_from_sim no)
+		(in_bom yes)
+		(on_board yes)
+		(in_pos_files yes)
+		(dnp no)
+		(property "Reference" "#PWR04"
+			(at 39.37 111.76 0)
+			(show_name no)
+			(do_not_autoplace no)
+			(effects
+				(font
+					(size 1.27 1.27)
+				)
+			)
+		)
+		(property "Value" "PWR_FLAG"
+			(at 39.37 116.84 0)
+			(show_name no)
+			(do_not_autoplace no)
+			(effects
+				(font
+					(size 1.27 1.27)
+				)
+			)
+		)
+		(property "Footprint" ""
+			(at 39.37 114.3 0)
+			(hide yes)
+			(show_name no)
+			(do_not_autoplace no)
+			(effects
+				(font
+					(size 1.27 1.27)
+				)
+			)
+		)
+		(property "Datasheet" ""
+			(at 39.37 114.3 0)
+			(hide yes)
+			(show_name no)
+			(do_not_autoplace no)
+			(effects
+				(font
+					(size 1.27 1.27)
+				)
+			)
+		)
+		(property "Description" "Special symbol for telling ERC where power comes from"
+			(at 39.37 114.3 0)
+			(hide yes)
+			(show_name no)
+			(do_not_autoplace no)
+			(effects
+				(font
+					(size 1.27 1.27)
+				)
+			)
+		)
+		(pin "1"
+		)
+		(instances
+			(project "receiver"
+				(path "/190c1e52-8c3e-49f8-9174-beae767bddea"
+					(reference "#PWR04")
+					(unit 1)
+				)
+			)
+		)
+	)
+	(label "VBUS"
+		(at 39.37 111.76 90)
+		(effects
+			(font
+				(size 1.27 1.27)
+			)
+			(justify left bottom)
+		)
+	)
+	(label "GND"
+		(at 39.37 114.3 90)
+		(effects
+			(font
+				(size 1.27 1.27)
+			)
+			(justify left bottom)
+		)
+	)

Commit message: devlog 04
Parts:
- C1, C2, C3: footprint (none) -> Capacitor_SMD:C_0603_1608Metric
- D1: footprint (none) -> LED_SMD:LED_0603_1608Metric
- HDR1: footprint (none) -> Connector_PinHeader_2.54mm:PinHeader_1x03_P2.54mm_Vertical
- J1: footprint (none) -> Connector_USB:USB_C_Receptacle_HRO_TYPE-C-31-M-12
- R_ACT, R_CC1, R_CC2, R_EN: footprint (none) -> Resistor_SMD:R_0603_1608Metric
- SW_BOOT, SW_RST: footprint (none) -> Button_Switch_SMD:SW_SPST_B3U-1000P
- U1: footprint (none) -> RF_Module:ESP32-S3-WROOM-1
- U2: footprint (none) -> Package_TO_SOT_SMD:SOT-23-5
Changed lines of the file:
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@@
 			)
 		)
-		(property "Footprint" ""
+		(property "Footprint" "Capacitor_SMD:C_0603_1608Metric"
 			(at 122.885 140.97 0)
 			(hide yes)
@@
 			)
 		)
-		(property "Footprint" ""
+		(property "Footprint" "Resistor_SMD:R_0603_1608Metric"
 			(at 68.072 80.01 90)
 			(hide yes)
@@
 			)
 		)
-		(property "Footprint" ""
+		(property "Footprint" "Capacitor_SMD:C_0603_1608Metric"
 			(at 107.645 140.97 0)
 			(hide yes)
@@
 			)
 		)
-		(property "Footprint" ""
+		(property "Footprint" "Connector_PinHeader_2.54mm:PinHeader_1x03_P2.54mm_Vertical"
 			(at 157.48 99.06 0)
 			(hide yes)
@@
 			)
 		)
-		(property "Footprint" ""
+		(property "Footprint" "Resistor_SMD:R_0603_1608Metric"
 			(at 93.472 74.93 90)
 			(hide yes)
@@
 			)
 		)
-		(property "Footprint" ""
+		(property "Footprint" "Package_TO_SOT_SMD:SOT-23-5"
 			(at 80.01 132.715 0)
 			(hide yes)
@@
 			)
 		)
-		(property "Footprint" ""
+		(property "Footprint" "Button_Switch_SMD:SW_SPST_B3U-1000P"
 			(at 165.1 165.1 0)
 			(hide yes)
@@
 			)
 		)
-		(property "Footprint" ""
+		(property "Footprint" "Capacitor_SMD:C_0603_1608Metric"
 			(at 60.655 91.44 0)
 			(hide yes)
@@
 			)
 		)
-		(property "Footprint" ""
+		(property "Footprint" "Resistor_SMD:R_0603_1608Metric"
 			(at 148.082 134.62 90)
 			(hide yes)
@@
 			)
 		)
-		(property "Footprint" ""
+		(property "Footprint" "Resistor_SMD:R_0603_1608Metric"
 			(at 68.072 59.69 90)
 			(hide yes)
@@
 			)
 		)
-		(property "Footprint" ""
+		(property "Footprint" "LED_SMD:LED_0603_1608Metric"
 			(at 149.86 119.38 0)
 			(hide yes)
@@
 			)
 		)
-		(property "Footprint" ""
+		(property "Footprint" "Button_Switch_SMD:SW_SPST_B3U-1000P"
 			(at 144.78 165.1 0)
 			(hide yes)
@@
 			)
 		)
-		(property "Footprint" ""
+		(property "Footprint" "Connector_USB:USB_C_Receptacle_HRO_TYPE-C-31-M-12"
 			(at 48.26 69.85 0)
 			(hide yes)
@@
 			)
 		)
-		(property "Footprint" ""
+		(property "Footprint" "RF_Module:ESP32-S3-WROOM-1"
 			(at 119.38 107.95 0)
 			(hide yes)
