File: receiver/receiver.kicad_pcb (KiCad board)
At the start: 2 copper layers, 0 parts

Commit message: devlog 04
Parts:
- added C1: 100nF, Capacitor_SMD:C_0603_1608Metric, F.Cu at (145.8, 111.2)
- added C2: 10uF, Capacitor_SMD:C_0603_1608Metric, F.Cu at (156.2, 109.7)
- added C3: 1uF, Capacitor_SMD:C_0603_1608Metric, F.Cu at (142.8, 111.2)
- added D1: ACT, LED_SMD:LED_0603_1608Metric, F.Cu at (139.8, 109.7)
- added HDR1: DEBUG, Connector_PinHeader_2.54mm:PinHeader_1x03_P2.54mm_Vertical, F.Cu at (156.2, 115.0)
- added J1: USB-C, Connector_USB:USB_C_Receptacle_HRO_TYPE-C-31-M-12, F.Cu at (148.3, 117.7)
- added R_ACT: 1k, Resistor_SMD:R_0603_1608Metric, F.Cu at (142.8, 109.7)
- added R_CC1: 5.1k, Resistor_SMD:R_0603_1608Metric, F.Cu at (141.6, 112.7)
- added R_CC2: 5.1k, Resistor_SMD:R_0603_1608Metric, F.Cu at (153.2, 109.8)
- added R_EN: 10k, Resistor_SMD:R_0603_1608Metric, F.Cu at (145.8, 109.7)
- added SW_BOOT: BOOT, Button_Switch_SMD:SW_SPST_B3U-1000P, F.Cu at (140.6, 116.8)
- added SW_RST: RESET, Button_Switch_SMD:SW_SPST_B3U-1000P, F.Cu at (140.6, 120.2)
- added U1: ESP32-S3-WROOM-1, RF_Module:ESP32-S3-WROOM-1, F.Cu at (148.1, 95.5)
- added U2: AP2112K-3.3, Package_TO_SOT_SMD:SOT-23-5, F.Cu at (149.6, 110.7)
Routing:
- net GND: track 0.00 -> 51.2 mm, vias 0 -> 6
- net 3v3: track 0.00 -> 41.8 mm, vias 0 -> 8
- net EN_NET: track 0.00 -> 39.2 mm, vias 0 -> 3
- net LED_ACT: track 0.00 -> 34.5 mm, vias 0 -> 2
- net UART_TX: track 0.00 -> 29.0 mm, vias 0 -> 1
- net BOOT_NET: track 0.00 -> 26.5 mm
- net UART_RX: track 0.00 -> 24.9 mm, vias 0 -> 1
- net USB_DP: track 0.00 -> 17.4 mm, vias 0 -> 2
- net USB_DN: track 0.00 -> 16.4 mm, vias 0 -> 2
- net VBUS: track 0.00 -> 15.4 mm
- net CC2: track 0.00 -> 7.99 mm, vias 0 -> 2
- net CC1: track 0.00 -> 6.80 mm, vias 0 -> 2
- net ACT_A: track 0.00 -> 1.39 mm
- added copper zone on B.Cu, net GND
- added copper zone on F.Cu, net GND
Other:
- board outline added: 19.8 x 33.1 mm

Commit message: devlog 05
Routing:
- net 3v3: vias 8 -> 7
Other:
- board size 19.8 x 33.1 mm -> 20.8 x 34.1 mm
Changed lines of the file:
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@@
 		)
+	)
+	(gr_arc
+		(start 137.7 88.85)
+		(mid 137.890381 88.390381)
+		(end 138.35 88.2)
+		(stroke
+			(width 0)
+			(type default)
+		)
+		(layer "Edge.Cuts")
 	)
 	(gr_line
-		(start 138.3 89.35)
-		(end 138.2 121.15)
-		(stroke
-			(width 0.05)
+		(start 137.7 121.65)
+		(end 137.7 88.85)
+		(stroke
+			(width 0)
+			(type default)
+		)
+		(layer "Edge.Cuts")
+	)
+	(gr_line
+		(start 138.35 88.2)
+		(end 157.85 88.2)
+		(stroke
+			(width 0)
 			(type default)
 		)
@@
 	)
 	(gr_arc
-		(start 138.3 89.35)
-		(mid 138.490381 88.890381)
-		(end 138.95 88.7)
-		(stroke
-			(width 0.05)
+		(start 138.35 122.3)
+		(mid 137.890381 122.109619)
+		(end 137.7 121.65)
+		(stroke
+			(width 0)
 			(type default)
 		)
@@
 	)
 	(gr_arc
-		(start 138.85 121.8)
-		(mid 138.390381 121.609619)
-		(end 138.2 121.15)
-		(stroke
-			(width 0.05)
+		(start 157.85 88.2)
+		(mid 158.309619 88.390381)
+		(end 158.5 88.85)
+		(stroke
+			(width 0)
 			(type default)
 		)
@@
 	)
 	(gr_line
-		(start 138.85 121.8)
-		(end 157.35 121.8)
-		(stroke
-			(width 0.05)
+		(start 157.85 122.3)
+		(end 138.35 122.3)
+		(stroke
+			(width 0)
 			(type default)
 		)
@@
 	)
 	(gr_line
-		(start 157.35 88.7)
-		(end 138.95 88.7)
-		(stroke
-			(width 0.05)
+		(start 158.5 88.85)
+		(end 158.5 121.65)
+		(stroke
+			(width 0)
 			(type default)
 		)
@@
 	)
 	(gr_arc
-		(start 157.35 88.7)
-		(mid 157.809619 88.890381)
-		(end 158 89.35)
-		(stroke
-			(width 0.05)
-			(type default)
-		)
-		(layer "Edge.Cuts")
-	)
-	(gr_arc
-		(start 158 121.15)
-		(mid 157.809619 121.609619)
-		(end 157.35 121.8)
-		(stroke
-			(width 0.05)
-			(type default)
-		)
-		(layer "Edge.Cuts")
-	)
-	(gr_line
-		(start 158 121.15)
-		(end 158 89.35)
-		(stroke
-			(width 0.05)
+		(start 158.5 121.65)
+		(mid 158.309619 122.109619)
+		(end 157.85 122.3)
+		(stroke
+			(width 0)
 			(type default)
 		)
@@
 		(size 0.6)
 		(drill 0.3)
-		(layers "F.Cu" "B.Cu")
-		(net "3v3")
-	)
-	(via
-		(at 154.95 110.35)
-		(size 0.6)
-		(drill 0.3)

Commit message: devlog 06
Other:
- board text added: "Designed by EVV"
- board text added: "Made for Hack Club Half Life"
Changed lines of the file:
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@@
 		(tags "resistor")
 		(property "Reference" "R_EN"
-			(at 0 -1.43 0)
+			(at 0.1 0.75 0)
 			(layer "F.SilkS")
 			(effects
@@
 		(tags "capacitor")
 		(property "Reference" "C3"
-			(at 0 -1.43 0)
+			(at 3.75 -1.1 0)
 			(layer "F.SilkS")
 			(effects
@@
 		(tags "Tactile Switch")
 		(property "Reference" "SW_RST"
-			(at 0 -2.5 0)
+			(at 0.1 1.55 0)
 			(layer "F.SilkS")
 			(effects
@@
 		(tags "LED")
 		(property "Reference" "D1"
-			(at 0 -1.43 0)
+			(at -0.9 1.25 0)
 			(layer "F.SilkS")
 			(effects
@@
 		(tags "2.4 GHz Wi-Fi and Bluetooth module")
 		(property "Reference" "U1"
-			(at -10.5 11.4 90)
+			(at -6.7 10.49 0)
 			(unlocked yes)
 			(layer "F.SilkS")
@@
 		(tags "capacitor")
 		(property "Reference" "C2"
-			(at 0 -1.43 0)
+			(at 1.1 1.4 0)
 			(layer "F.SilkS")
 			(effects
@@
 		(tags "usb usb-c 2.0 pd")
 		(property "Reference" "J1"
-			(at 0 -5.645 0)
+			(at -1.45 -5.36 0)
 			(layer "F.SilkS")
 			(effects
@@
 		(tags "capacitor")
 		(property "Reference" "C1"
-			(at 0 -1.43 0)
+			(at -0.625 1.15 0)
 			(layer "F.SilkS")
 			(effects
@@
 		(tags "resistor")
 		(property "Reference" "R_CC1"
-			(at 0 -1.43 0)
+			(at 1.25 -0.95 0)
 			(layer "F.SilkS")
 			(effects
@@
 		(tags "SOT TO_SOT_SMD")
 		(property "Reference" "U2"
-			(at 0 -2.4 0)
+			(at 0.6625 0 0)
 			(layer "F.SilkS")
 			(effects
@@
 		(tags "resistor")
 		(property "Reference" "R_ACT"
-			(at 0 -1.43 0)
+			(at 0.9 -0.75 0)
 			(layer "F.SilkS")
 			(effects
@@
 		(tags "resistor")
 		(property "Reference" "R_CC2"
-			(at 0 -1.43 0)
+			(at 0.725 1.25 0)
 			(layer "F.SilkS")
 			(effects
@@
 		(tags "Tactile Switch")
 		(property "Reference" "SW_BOOT"
-			(at 0 -2.5 0)
+			(at -0.2 -2.15 0)
 			(layer "F.SilkS")
 			(effects
 				(font
-					(size 1 1)
+					(size 0.8 0.8)
 					(thickness 0.15)
 				)
@@
 		(end 138.35 88.2)
 		(stroke
-			(width 0)
+			(width 0.1)
 			(type default)
 		)
@@
 		(end 137.7 88.85)
 		(stroke
-			(width 0)
+			(width 0.1)
 			(type default)
 		)
@@
 		(end 157.85 88.2)
 		(stroke
-			(width 0)
+			(width 0.1)
 			(type default)
 		)
@@
 		(end 137.7 121.65)
 		(stroke
-			(width 0)
+			(width 0.1)
 			(type default)
 		)
@@
 		(end 158.5 88.85)
 		(stroke
-			(width 0)
+			(width 0.1)
 			(type default)
 		)
@@
 		(end 138.35 122.3)
 		(stroke
-			(width 0)
+			(width 0.1)
 			(type default)
 		)
@@
 		(end 158.5 121.65)
 		(stroke
-			(width 0)
+			(width 0.1)
 			(type default)
 		)
@@
 		(end 157.85 122.3)
 		(stroke
-			(width 0)
+			(width 0.1)
 			(type default)
 		)
 		(layer "Edge.Cuts")
 	)
+	(gr_text "Made for Hack Club Half Life"
+		(at 153.4 91.25 -0)
+		(layer "B.SilkS")
+		(effects
+			(font
+				(size 0.5 0.5)
+				(thickness 0.1)
+			)
+			(justify left bottom mirror)
+		)
+	)
+	(gr_text "Designed by EVV"
+		(at 154.1 90.05 -0)
+		(layer "B.SilkS")
+		(effects
+			(font
+				(size 1 1)
+				(thickness 0.15)
+			)
+			(justify left bottom mirror)
+		)
+	)
 	(segment
